Commit message: fix fr3.urdf

File: model/franka_emika_panda/fr3.urdf (robot description, URDF)
Before this commit: robot panda, 12 links, 11 joints
Links:
- link panda_hand: geometry 
- link panda_leftfinger: geometry 
- link panda_link0: geometry 
- link panda_link1: geometry 
- link panda_link2: geometry 
- link panda_link3: geometry 
- link panda_link4: geometry 
- link panda_link5: geometry 
- link panda_link6: geometry 
- link panda_link7: geometry 
- link panda_rightfinger: geometry 
